Commit message: Add source folder for Gazebo simulation

File: src/Universal_Robots_ROS2_Description/urdf/ur_macro.xacro (robot description, xacro)
@@ -356,5 +356,5 @@
       <dynamics damping="0" friction="0"/>
     </joint>
-    <link name="${tf_prefix}bowl_link">
+    <!-- <link name="${tf_prefix}bowl_link">
       <visual>
         <origin xyz="0 0 0" rpy="0 0 0"/>
@@ -378,5 +378,5 @@
       <child link="${tf_prefix}bowl_link"/>
       <origin xyz="0 0 0" rpy="0 0 0"/>
-    </joint>
+    </joint> -->
     <link name="${tf_prefix}ft_frame"/>
     <joint name="${tf_prefix}wrist_3_link-ft_frame" type="fixed">
@@ -403,4 +403,17 @@
       <child link="${tf_prefix}tool0"/>
     </joint>
+    <gazebo reference="wrist_3_link">
+      <sensor type="force_torque" name="wrist_ft_sensor">
+        <always_on>1</always_on>
+        <update_rate>100</update_rate>
+        <pose>0 0 0 0 0 0</pose>
+        <plugin name="gazebo_ros_ft_sensor" filename="libgazebo_ros_ft_sensor.so">
+          <robotNamespace>/ur10e</robotNamespace>
+          <jointName>wrist_3_joint</jointName>
+          <topicName>/ur10e/wrist_ft/wrench</topicName>
+          <frameName>wrist_3_link</frameName>
+        </plugin>
+      </sensor>
+    </gazebo>
   </xacro:macro>
 </robot>

Commit message: Updated cartesian planning code

File: src/Universal_Robots_ROS2_Description/urdf/ur_macro.xacro (robot description, xacro)
@@ -1,4 +1,45 @@
 <?xml version="1.0"?>
 <robot xmlns:xacro="http://wiki.ros.org/xacro">
+  <!--
+    Base UR robot series xacro macro.
+    NOTE this is NOT a URDF. It cannot directly be loaded by consumers
+    expecting a flattened '.urdf' file. See the top-level '.xacro' for that
+    (but note that .xacro must still be processed by the xacro command).
+    This file models the base kinematic chain of a UR robot, which then gets
+    parameterised by various configuration files to convert it into a UR3(e),
+    UR5(e), UR10(e) or UR16e, etc.
+    NOTE the default kinematic parameters (i.e., link lengths, frame locations,
+    offsets, etc) do not correspond to any particular robot. They are defaults
+    only. There WILL be non-zero offsets between the Forward Kinematics results
+    in TF (i.e., robot_state_publisher) and the values reported by the Teach
+    Pendant.
+    For accurate (and robot-specific) transforms, the 'kinematics_parameters_file'
+    parameter MUST point to a .yaml file containing the appropriate values for
+    the targeted robot.
+    If using the UniversalRobots/Universal_Robots_ROS_Driver, follow the steps
+    described in the readme of that repository to extract the kinematic
+    calibration from the controller and generate the required .yaml file.
+    Main author of the migration to yaml configs Ludovic Delval.
+    Contributors to previous versions (in no particular order)
+     - Denis Stogl
+     - Lovro Ivanov
+     - Felix Messmer
+     - Kelsey Hawkins
+     - Wim Meeussen
+     - Shaun Edwards
+     - Nadia Hammoudeh Garcia
+     - Dave Hershberger
+     - G. vd. Hoorn
+     - Philip Long
+     - Dave Coleman
+     - Miguel Prada
+     - Mathias Luedtke
+     - Marcel Schnirring
+     - Felix von Drigalski
+     - Felix Exner
+     - Jimmy Da Silva
+     - Ajit Krisshna N L
+     - Muhammad Asif Rana
+  -->
   <xacro:include filename="$(find ur_description)/urdf/inc/ur_transmissions.xacro" />
   <xacro:include filename="$(find ur_description)/urdf/inc/ur_common.xacro" />
@@ -44,4 +85,5 @@
     keep_alive_count:=2"
     >
+    <!-- Load configuration data from the provided .yaml files -->
     <xacro:read_model_data
       joint_limits_parameters_file="${joint_limits_parameters_file}"
@@ -51,5 +93,7 @@
       force_abs_paths="${sim_gazebo or sim_ignition}"/>
     <xacro:if value="${generate_ros2_control_tag}">
+      <!-- ros2 control include -->
       <xacro:include filename="$(find ur_description)/urdf/ur.ros2_control.xacro" />
+      <!-- ros2 control instance -->
       <xacro:ur_ros2_control
         name="${name}"
@@ -82,6 +126,10 @@
         non_blocking_read="${non_blocking_read}"
         keep_alive_count="${keep_alive_count}"
-      />
+        />
     </xacro:if>
+    <!-- Add URDF transmission elements (for ros_control) -->
+    <!--<xacro:ur_arm_transmission prefix="${prefix}" hw_interface="${transmission_hw_interface}" />-->
+    <!-- Placeholder for ros2_control transmission which don't yet exist -->
+    <!-- links -  main serial chain -->
     <link name="${tf_prefix}base_link"/>
     <link name="${tf_prefix}base_link_inertia">
@@ -119,13 +167,12 @@
         <origin rpy="${shoulder_inertia_rotation}" xyz="${shoulder_cog}"/>
         <inertia
-          ixx="${shoulder_inertia_ixx}"
-          ixy="${shoulder_inertia_ixy}"
-          ixz="${shoulder_inertia_ixz}"
-          iyy="${shoulder_inertia_iyy}"
-          iyz="${shoulder_inertia_iyz}"
-          izz="${shoulder_inertia_izz}"
-        />
-      </inertial>
-    </link>
+            ixx="${shoulder_inertia_ixx}"
+            ixy="${shoulder_inertia_ixy}"
+            ixz="${shoulder_inertia_ixz}"
+            iyy="${shoulder_inertia_iyy}"
+            iyz="${shoulder_inertia_iyz}"
+            izz="${shoulder_inertia_izz}"
+        />
+      </inertial>    </link>
     <link name="${tf_prefix}upper_arm_link">
       <visual>
@@ -145,10 +192,10 @@
         <origin rpy="${upper_arm_inertia_rotation}" xyz="${upper_arm_cog}"/>
         <inertia
-          ixx="${upper_arm_inertia_ixx}"
-          ixy="${upper_arm_inertia_ixy}"
-          ixz="${upper_arm_inertia_ixz}"
-          iyy="${upper_arm_inertia_iyy}"
-          iyz="${upper_arm_inertia_iyz}"
-          izz="${upper_arm_inertia_izz}"
+            ixx="${upper_arm_inertia_ixx}"
+            ixy="${upper_arm_inertia_ixy}"
+            ixz="${upper_arm_inertia_ixz}"
+            iyy="${upper_arm_inertia_iyy}"
+            iyz="${upper_arm_inertia_iyz}"
+            izz="${upper_arm_inertia_izz}"
         />
       </inertial>
@@ -171,17 +218,17 @@
         <origin rpy="${forearm_inertia_rotation}" xyz="${forearm_cog}"/>
         <inertia
-          ixx="${forearm_inertia_ixx}"
-          ixy="${forearm_inertia_ixy}"
-          ixz="${forearm_inertia_ixz}"
-          iyy="${forearm_inertia_iyy}"
-          iyz="${forearm_inertia_iyz}"
-          izz="${forearm_inertia_izz}"
+            ixx="${forearm_inertia_ixx}"
+            ixy="${forearm_inertia_ixy}"
+            ixz="${forearm_inertia_ixz}"
+            iyy="${forearm_inertia_iyy}"
+            iyz="${forearm_inertia_iyz}"
+            izz="${forearm_inertia_izz}"
         />
       </inertial>
     </link>
     <link name="${tf_prefix}wrist_1_link">
-      <xacro:get_visual_params name="wrist_1" type="visual_offset"/>
-      <visual>
-        <origin xyz="0 0 ${visual_params}" rpy="${pi/2} 0 0"/>
+	  <xacro:get_visual_params name="wrist_1" type="visual_offset"/>
+      <visual>
+      	<origin xyz="0 0 ${visual_params}" rpy="${pi/2} 0 0"/>
         <geometry>
           <xacro:get_mesh name="wrist_1" type="visual"/>
@@ -198,15 +245,15 @@
         <origin rpy="${wrist_1_inertia_rotation}" xyz="${wrist_1_cog}"/>
         <inertia
-          ixx="${wrist_1_inertia_ixx}"
-          ixy="${wrist_1_inertia_ixy}"
-          ixz="${wrist_1_inertia_ixz}"
-          iyy="${wrist_1_inertia_iyy}"
-          iyz="${wrist_1_inertia_iyz}"
-          izz="${wrist_1_inertia_izz}"
+            ixx="${wrist_1_inertia_ixx}"
+            ixy="${wrist_1_inertia_ixy}"
+            ixz="${wrist_1_inertia_ixz}"
+            iyy="${wrist_1_inertia_iyy}"
+            iyz="${wrist_1_inertia_iyz}"
+            izz="${wrist_1_inertia_izz}"
         />
       </inertial>
     </link>
     <link name="${tf_prefix}wrist_2_link">
-      <xacro:get_visual_params name="wrist_2" type="visual_offset"/>
+          <xacro:get_visual_params name="wrist_2" type="visual_offset"/>
       <visual>
         <origin xyz="0 0 ${visual_params}" rpy="0 0 0"/>
@@ -225,14 +272,15 @@
         <origin rpy="${wrist_2_inertia_rotation}" xyz="${wrist_2_cog}"/>
         <inertia
-          ixx="${wrist_2_inertia_ixx}"
-          ixy="${wrist_2_inertia_ixy}"
-          ixz="${wrist_2_inertia_ixz}"
-          iyy="${wrist_2_inertia_iyy}"
-          iyz="${wrist_2_inertia_iyz}"
-          izz="${wrist_2_inertia_izz}"
+            ixx="${wrist_2_inertia_ixx}"
+            ixy="${wrist_2_inertia_ixy}"
+            ixz="${wrist_2_inertia_ixz}"
+            iyy="${wrist_2_inertia_iyy}"
+            iyz="${wrist_2_inertia_iyz}"
+            izz="${wrist_2_inertia_izz}"
         />
       </inertial>
     </link>
     <link name="${tf_prefix}wrist_3_link">
+      <!-- TODO: remove this once all wrist_3 meshes have the visual_offset_xyz tag -->
       <xacro:get_visual_params name="wrist_3" type="visual_offset_xyz"/>
       <xacro:property name="mesh_offset" value="${visual_params}" scope="parent"/>
@@ -257,13 +305,14 @@
         <origin rpy="${wrist_3_inertia_rotation}" xyz="${wrist_3_cog}"/>
         <inertia
-          ixx="${wrist_3_inertia_ixx}"
-          ixy="${wrist_3_inertia_ixy}"
-          ixz="${wrist_3_inertia_ixz}"
-          iyy="${wrist_3_inertia_iyy}"
-          iyz="${wrist_3_inertia_iyz}"
-          izz="${wrist_3_inertia_izz}"
+            ixx="${wrist_3_inertia_ixx}"
+            ixy="${wrist_3_inertia_ixy}"
+            ixz="${wrist_3_inertia_ixz}"
+            iyy="${wrist_3_inertia_iyy}"
+            iyz="${wrist_3_inertia_iyz}"
+            izz="${wrist_3_inertia_izz}"
         />
       </inertial>
     </link>
+    <!-- base_joint fixes base_link to the environment -->
     <joint name="${tf_prefix}base_joint" type="fixed">
       <xacro:insert_block name="origin" />
@@ -271,7 +320,13 @@
       <child link="${tf_prefix}base_link" />
     </joint>
+    <!-- joints - main serial chain -->
     <joint name="${tf_prefix}base_link-base_link_inertia" type="fixed">
       <parent link="${tf_prefix}base_link" />
       <child link="${tf_prefix}base_link_inertia" />
+      <!-- 'base_link' is REP-103 aligned (so X+ forward), while the internal
+           frames of the robot/controller have X+ pointing backwards.
+           Use the joint between 'base_link' and 'base_link_inertia' (a dummy
+           link/frame) to introduce the necessary rotation over Z (of pi rad).
+      -->
       <origin xyz="0 0 0" rpy="0 0 ${pi}" />
     </joint>
@@ -284,5 +339,5 @@
         effort="${shoulder_pan_effort_limit}" velocity="${shoulder_pan_velocity_limit}"/>
       <xacro:if value="${safety_limits}">
-        <safety_controller soft_lower_limit="${shoulder_pan_lower_limit + safety_pos_margin}" soft_upper_limit="${shoulder_pan_upper_limit - safety_pos_margin}" k_position="${safety_k_position}" k_velocity="0.0"/>
+         <safety_controller soft_lower_limit="${shoulder_pan_lower_limit + safety_pos_margin}" soft_upper_limit="${shoulder_pan_upper_limit - safety_pos_margin}" k_position="${safety_k_position}" k_velocity="0.0"/>
       </xacro:if>
       <dynamics damping="0" friction="0"/>
@@ -296,5 +351,5 @@
         effort="${shoulder_lift_effort_limit}" velocity="${shoulder_lift_velocity_limit}"/>
       <xacro:if value="${safety_limits}">
-        <safety_controller soft_lower_limit="${shoulder_lift_lower_limit + safety_pos_margin}" soft_upper_limit="${shoulder_lift_upper_limit - safety_pos_margin}" k_position="${safety_k_position}" k_velocity="0.0"/>
+         <safety_controller soft_lower_limit="${shoulder_lift_lower_limit + safety_pos_margin}" soft_upper_limit="${shoulder_lift_upper_limit - safety_pos_margin}" k_position="${safety_k_position}" k_velocity="0.0"/>
       </xacro:if>
       <dynamics damping="0" friction="0"/>
@@ -308,5 +363,5 @@
         effort="${elbow_joint_effort_limit}" velocity="${elbow_joint_velocity_limit}"/>
       <xacro:if value="${safety_limits}">
-        <safety_controller soft_lower_limit="${elbow_joint_lower_limit + safety_pos_margin}" soft_upper_limit="${elbow_joint_upper_limit - safety_pos_margin}" k_position="${safety_k_position}" k_velocity="0.0"/>
+         <safety_controller soft_lower_limit="${elbow_joint_lower_limit + safety_pos_margin}" soft_upper_limit="${elbow_joint_upper_limit - safety_pos_margin}" k_position="${safety_k_position}" k_velocity="0.0"/>
       </xacro:if>
       <dynamics damping="0" friction="0"/>
@@ -320,5 +375,5 @@
         effort="${wrist_1_effort_limit}" velocity="${wrist_1_velocity_limit}"/>
       <xacro:if value="${safety_limits}">
-        <safety_controller soft_lower_limit="${wrist_1_lower_limit + safety_pos_margin}" soft_upper_limit="${wrist_1_upper_limit - safety_pos_margin}" k_position="${safety_k_position}" k_velocity="0.0"/>
+         <safety_controller soft_lower_limit="${wrist_1_lower_limit + safety_pos_margin}" soft_upper_limit="${wrist_1_upper_limit - safety_pos_margin}" k_position="${safety_k_position}" k_velocity="0.0"/>
       </xacro:if>
       <dynamics damping="0" friction="0"/>
@@ -332,5 +387,5 @@
              effort="${wrist_2_effort_limit}" velocity="${wrist_2_velocity_limit}"/>
       <xacro:if value="${safety_limits}">
-        <safety_controller soft_lower_limit="${wrist_2_lower_limit + safety_pos_margin}" soft_upper_limit="${wrist_2_upper_limit - safety_pos_margin}" k_position="${safety_k_position}" k_velocity="0.0"/>
+         <safety_controller soft_lower_limit="${wrist_2_lower_limit + safety_pos_margin}" soft_upper_limit="${wrist_2_upper_limit - safety_pos_margin}" k_position="${safety_k_position}" k_velocity="0.0"/>
       </xacro:if>
       <dynamics damping="0" friction="0"/>
@@ -356,27 +411,4 @@
       <dynamics damping="0" friction="0"/>
     </joint>
-    <!-- <link name="${tf_prefix}bowl_link">
-      <visual>
-        <origin xyz="0 0 0" rpy="0 0 0"/>
-        <geometry>
-          <mesh filename="package://ur_description/meshes/ur10e/collision/bowl.stl" scale="0.002 0.002 0.002"/>
-        </geometry>
-      </visual>
-      <collision>
-        <origin xyz="0 0 0" rpy="0 0 0"/>
-        <geometry>
-          <mesh filename="package://ur_description/meshes/ur10e/collision/bowl.stl" scale="0.002 0.002 0.002"/>
-        </geometry>
-      </collision>
-      <inertial>
-        <mass value="0.1"/>
-        <inertia ixx="0.001" ixy="0" ixz="0" iyy="0.001" iyz="0" izz="0.001"/>
-      </inertial>
-    </link>
-    <joint name="${tf_prefix}base_to_bowl_joint" type="fixed">
-      <parent link="${tf_prefix}base_link"/>
-      <child link="${tf_prefix}bowl_link"/>
-      <origin xyz="0 0 0" rpy="0 0 0"/>
-    </joint> -->
     <link name="${tf_prefix}ft_frame"/>
     <joint name="${tf_prefix}wrist_3_link-ft_frame" type="fixed">
@@ -385,10 +417,17 @@
       <origin xyz="0 0 0" rpy="${pi} 0 0"/>
     </joint>
+    <!-- ROS-Industrial 'base' frame - base_link to UR 'Base' Coordinates transform -->
     <link name="${tf_prefix}base"/>
     <joint name="${tf_prefix}base_link-base_fixed_joint" type="fixed">
+      <!-- Note the rotation over Z of pi radians - as base_link is REP-103
+           aligned (i.e., has X+ forward, Y+ left and Z+ up), this is needed
+           to correctly align 'base' with the 'Base' coordinate system of
+           the UR controller.
+      -->
       <origin xyz="0 0 0" rpy="0 0 ${pi}"/>
       <parent link="${tf_prefix}base_link"/>
       <child link="${tf_prefix}base"/>
     </joint>
+    <!-- ROS-Industrial 'flange' frame - attachment point for EEF models -->
     <link name="${tf_prefix}flange" />
     <joint name="${tf_prefix}wrist_3-flange" type="fixed">
@@ -397,23 +436,12 @@
       <origin xyz="0 0 0" rpy="0 ${-pi/2.0} ${-pi/2.0}" />
     </joint>
+    <!-- ROS-Industrial 'tool0' frame - all-zeros tool frame -->
     <link name="${tf_prefix}tool0"/>
     <joint name="${tf_prefix}flange-tool0" type="fixed">
+      <!-- default toolframe - X+ left, Y+ up, Z+ front -->
       <origin xyz="0 0 0" rpy="${pi/2.0} 0 ${pi/2.0}"/>
       <parent link="${tf_prefix}flange"/>
       <child link="${tf_prefix}tool0"/>
     </joint>
-    <gazebo reference="wrist_3_link">
-      <sensor type="force_torque" name="wrist_ft_sensor">
-        <always_on>1</always_on>
-        <update_rate>100</update_rate>
-        <pose>0 0 0 0 0 0</pose>
-        <plugin name="gazebo_ros_ft_sensor" filename="libgazebo_ros_ft_sensor.so">
-          <robotNamespace>/ur10e</robotNamespace>
-          <jointName>wrist_3_joint</jointName>
-          <topicName>/ur10e/wrist_ft/wrench</topicName>
-          <frameName>wrist_3_link</frameName>
-        </plugin>
-      </sensor>
-    </gazebo>
   </xacro:macro>
 </robot>
