Commit message: Add mixer + UR10e combined Gazebo workspace updates

File: ur10e_simulation_pkg/urdf/vertical_mixer_planetary.urdf (robot description, URDF)
Before this commit: robot planetary_mixer, 8 links, 7 joints
Links:
- link base_link: mass 2.0 -> 50.0; geometry collision cylinder length=0.60 radius=0.30; visual mesh filename=package://ur10e_simulation_pkg/meshes/structure.stl scale=1 1 1
- link planet_1_carrier: mass 0.2 -> 0.001; geometry 
- link planet_1_link: mass 0.1 -> 1.5; geometry collision cylinder length=0.25 radius=0.045; visual mesh filename=package://ur10e_simulation_pkg/meshes/blade_1.stl scale=1 1 1
- link planet_2_carrier: mass 0.2 -> 0.001; geometry 
- link planet_2_link: mass 0.1 -> 1.5; geometry collision cylinder length=0.25 radius=0.045; visual mesh filename=package://ur10e_simulation_pkg/meshes/blade_2.stl scale=1 1 1
- link shroud_link: mass 1.0 -> 3.0; geometry collision cylinder length=0.40 radius=0.18; visual mesh filename=package://ur10e_simulation_pkg/meshes/shroud.stl scale=1 1 1
- link sun_link: mass 0.5 -> 2.0; geometry collision cylinder length=0.25 radius=0.06; visual mesh filename=package://ur10e_simulation_pkg/meshes/middle_blade.stl scale=1 1 1
Joints:
- joint planet_1_orbit_joint: origin xyz=0 0 0.025 rpy=0 0 0 -> xyz=0 0 0 rpy=0 0 0
- joint planet_1_spin_joint: origin xyz=0.08 0 0.02 rpy=0 0 0 -> xyz=0.155943 -0.456764 0 rpy=0 0 0
- joint planet_2_orbit_joint: origin xyz=0 0 0.025 rpy=0 0 3.14159265 -> xyz=0 0 0 rpy=0 0 0
- joint planet_2_spin_joint: origin xyz=0.08 0 0.02 rpy=0 0 0 -> xyz=-0.155847 0.456481 0 rpy=0 0 0
- joint shroud_joint: origin xyz=0 0 0.025 rpy=0 0 0 -> xyz=0 0 0 rpy=0 0 0
- joint sun_joint: origin xyz=0 0 0.025 rpy=0 0 0 -> xyz=0 0 0 rpy=0 0 0
