Commit message: Update UR10e force control and simulation vertical_mixer

File: Universal_Robots_ROS2_Description/urdf/ur_macro.xacro (robot description, xacro)
@@ -417,4 +417,76 @@
       <origin xyz="0 0 0" rpy="${pi} 0 0"/>
     </joint>
+    <!-- Wrist-mounted depth camera (D435i-like) -->
+    <link name="${tf_prefix}camera_link">
+      <inertial>
+        <origin xyz="0 0 0" rpy="0 0 0"/>
+        <mass value="0.072"/>
+        <inertia ixx="0.00002" ixy="0.0" ixz="0.0" iyy="0.00002" iyz="0.0" izz="0.00002"/>
+      </inertial>
+      <visual>
+        <origin xyz="0 0 0" rpy="0 0 0"/>
+        <geometry>
+          <box size="0.090 0.025 0.025"/>
+        </geometry>
+        <material name="camera_gray">
+          <color rgba="0.2 0.2 0.2 1.0"/>
+        </material>
+      </visual>
+      <collision>
+        <origin xyz="0 0 0" rpy="0 0 0"/>
+        <geometry>
+          <box size="0.090 0.025 0.025"/>
+        </geometry>
+      </collision>
+    </link>
+    <joint name="${tf_prefix}wrist_3-camera_joint" type="fixed">
+      <parent link="${tf_prefix}tool0"/>
+      <child link="${tf_prefix}camera_link"/>
+      <!-- Above wrist_3 and aligned so optical Z points dead-straight with tool forward -->
+      <origin xyz="0 0.07 0" rpy="${0} ${-pi/2.0} 0"/>
+    </joint>
+    <link name="${tf_prefix}camera_optical_frame"/>
+    <joint name="${tf_prefix}camera_optical_joint" type="fixed">
+      <parent link="${tf_prefix}camera_link"/>
+      <child link="${tf_prefix}camera_optical_frame"/>
+      <origin xyz="0 0 0" rpy="${-pi/2.0} 0 ${-pi/2.0}"/>
+    </joint>
+    <gazebo reference="${tf_prefix}camera_link">
+      <sensor name="${tf_prefix}depth_camera" type="depth">
+        <always_on>true</always_on>
+        <update_rate>30.0</update_rate>
+        <visualize>true</visualize>
+        <camera>
+          <horizontal_fov>1.396</horizontal_fov>
+          <image>
+            <width>640</width>
+            <height>480</height>
+            <format>R8G8B8</format>
+          </image>
+          <clip>
+            <near>0.1</near>
+            <far>5.0</far>
+          </clip>
+          <!-- Add gaussian depth noise so /camera/points has realistic sensor noise -->
+          <noise>
+            <type>gaussian</type>
+            <mean>0.0</mean>
+            <stddev>0.002</stddev>
+          </noise>
+          <depth_camera>
+            <clip>
+              <near>0.1</near>
+              <far>5.0</far>
+            </clip>
+          </depth_camera>
+        </camera>
+        <plugin name="${tf_prefix}depth_camera_controller" filename="libgazebo_ros_camera.so">
+          <camera_name>camera</camera_name>
+          <frame_name>${tf_prefix}camera_optical_frame</frame_name>
+          <min_depth>0.1</min_depth>
+          <max_depth>5.0</max_depth>
+        </plugin>
+      </sensor>
+    </gazebo>
     <link name="${tf_prefix}end_effector_link">
       <!-- ================= INERTIAL ================= -->

File: ur10e_simulation_pkg/urdf/vertical_mixer_planetary.urdf (robot description, URDF)
Before this commit: robot vertical_planetary_mixer, 8 links, 7 joints
Links:
- link base_link: geometry collision mesh filename=package://ur10e_simulation_pkg/meshes/structure.stl scale=1 1 1; visual mesh filename=package://ur10e_simulation_pkg/meshes/structure.stl scale=1 1 1
- link planet_1_link: geometry collision mesh filename=package://ur10e_simulation_pkg/meshes/blade_1.stl scale=1 1 1; visual mesh filename=package://ur10e_simulation_pkg/meshes/blade_1.stl scale=1 1 1
- link planet_2_link: geometry collision mesh filename=package://ur10e_simulation_pkg/meshes/blade_2.stl scale=1 1 1; visual mesh filename=package://ur10e_simulation_pkg/meshes/blade_2.stl scale=1 1 1
- link shroud_link: geometry collision mesh filename=package://ur10e_simulation_pkg/meshes/shroud.stl scale=1 1 1; visual mesh filename=package://ur10e_simulation_pkg/meshes/shroud.stl scale=1 1 1
- link sun_link: geometry collision mesh filename=package://ur10e_simulation_pkg/meshes/middle_blade.stl scale=1 1 1; visual mesh filename=package://ur10e_simulation_pkg/meshes/middle_blade.stl scale=1 1 1
